Commit message: Imu data simulation enhanced and linked the same in fourwd_robot.urdf

File: src/fourwd_robot/urdf/fourwd_robot.urdf (robot description, URDF)
Before this commit: robot fourwd_robot, 5 links, 4 joints
Links:
- added link imu_link; visual box size=0.06 0.03 0.05
- added link lidar_link; visual cylinder length=0.05 radius=0.05
Joints:
- added joint imu_joint: type fixed, parent base_link, child imu_link, origin xyz=0 0 0.1 rpy=0 1.57 0
- added joint lidar_joint: type fixed, parent base_link, child lidar_link, origin xyz=0.18 0 0.12 rpy=0 0 0

Commit message: Added xacro for the fourwd_robot

File: src/fourwd_robot/urdf/fourwd_robot.urdf (robot description, URDF)
Before this commit: robot fourwd_robot, 7 links, 6 joints
Joints:
- joint fl_wheel_joint: origin xyz=0.18  0.15 -0.065 rpy=0 0 0 -> xyz=0.18  0.167 0.034 rpy=0 0 0
- joint fr_wheel_joint: origin xyz=0.18 -0.15 -0.065 rpy=0 0 0 -> xyz=0.18 -0.167 0.034 rpy=0 0 0
- joint imu_joint: origin xyz=0 0 0.1 rpy=0 1.57 0 -> xyz=0 0 0.1 rpy=1.57 0 0
- joint rl_wheel_joint: origin xyz=-0.18  0.15 -0.065 rpy=0 0 0 -> xyz=-0.18  0.15 0.034 rpy=0 0 0
- joint rr_wheel_joint: origin xyz=-0.18 -0.15 -0.065 rpy=0 0 0 -> xyz=-0.18 -0.15 0.034 rpy=0 0 0
