Commit message: Fixed Rviz robot visulization

File: src/fourwd_robot/urdf/fourwd_robot.xacro (robot description, xacro)
@@ -30,4 +30,16 @@
         <material name="black"/>
       </visual>
+      <!--  Added collision props-->
+      <collision>
+      <origin xyz="0 0 0" rpy="1.5708 0 0"/>
+        <geometry>
+          <cylinder radius="${wheel_radius}" length="${wheel_width}"/>
+        </geometry>
+      </collision>
+      <!--  Added inertia props-->
+      <inertial>
+        <mass value="2.5"/>
+        <inertia ixx="0.15" ixy="0" ixz="0" iyy="0.15" iyz="0" izz="0.25"/>
+      </inertial>
     </link>
     <joint name="${prefix}_wheel_joint" type="continuous">
@@ -39,4 +51,12 @@
   </xacro:macro>
   <!-- ====================== BASE (CHASSIS) ====================== -->
+  <!-- ====================== DUMMY ROOT LINK (Massless) ====================== -->
+  <link name="base_footprint"/>
+  <!-- Fixed joint connecting dummy root to actual chassis -->
+  <joint name="base_footprint_to_base_link" type="fixed">
+    <parent link="base_footprint"/>
+    <child link="base_link"/>
+    <origin xyz="0 0 0" rpy="0 0 0"/>
+  </joint>
   <link name="base_link">
     <visual>
@@ -47,4 +67,16 @@
       <material name="blue"/>
     </visual>
+    <!-- Collision -->
+    <collision>
+      <origin xyz="0 0 ${chassis_height/2}" rpy="0 0 0"/>
+      <geometry>
+        <box size="${chassis_length} ${chassis_width} ${chassis_height}"/>
+      </geometry>
+    </collision>
+    <!-- Inertia  -->
+    <inertial>
+      <mass value="20.0"/>
+      <inertia ixx="2.0" ixy="0" ixz="0" iyy="1.8" iyz="0" izz="2.5"/>
+    </inertial>
   </link>
   <!-- ====================== WHEELS ====================== -->
@@ -67,4 +99,11 @@
       <material name="black"/>
     </visual>
+    <collision>
+      <geometry><cylinder length="0.05" radius="0.05"/></geometry>
+    </collision>
+    <inertial>
+      <mass value="0.5"/>
+      <inertia ixx="0.01" ixy="0" ixz="0" iyy="0.01" iyz="0" izz="0.01"/>
+    </inertial>
   </link>
   <joint name="lidar_joint" type="fixed">
@@ -73,4 +112,56 @@
     <origin xyz="0.18 0 0.1" rpy="0 0 0"/>
   </joint>
+  <!-- ====================== ROS2_CONTROL ====================== -->
+  <ros2_control name="GazeboSystem" type="system">
+     <hardware>
+        <plugin>mock_components/GenericSystem</plugin>
+        <params name="calculate_dynamics">true</params>
+    </hardware>
+    <joint name="fl_wheel_joint">
+      <command_interface name="velocity"/>
+      <state_interface name="velocity"/>
+      <state_interface name="position"/>
+    </joint>
+    <joint name="fr_wheel_joint">
+      <command_interface name="velocity"/>
+      <state_interface name="velocity"/>
+      <state_interface name="position"/>
+    </joint>
+    <joint name="rl_wheel_joint">
+      <command_interface name="velocity"/>
+      <state_interface name="velocity"/>
+      <state_interface name="position"/>
+    </joint>
+    <joint name="rr_wheel_joint">
+      <command_interface name="velocity"/>
+      <state_interface name="velocity"/>
+      <state_interface name="position"/>
+    </joint>
+  </ros2_control>
+   <!-- Gazebo LiDAR Plugin (GPU Ray Sensor) -->
+  <gazebo reference="lidar_link">
+    <sensor name="lidar_sensor" type="gpu_lidar">
+      <pose>0 0 0 0 0 0</pose>
+      <update_rate>20</update_rate>
+      <topic>scan</topic>
+      <always_on>true</always_on>
+      <visualize>true</visualize>
+      <ray>
+        <scan>
+          <horizontal>
+            <samples>720</samples>
+            <resolution>1</resolution>
+            <min_angle>-3.14159</min_angle>
+            <max_angle>3.14159</max_angle>
+          </horizontal>
+        </scan>
+        <range>
+          <min>0.1</min>
+          <max>30.0</max>
+          <resolution>0.01</resolution>
+        </range>
+      </ray>
+    </sensor>
+  </gazebo>
   <!-- IMU center-top -->
   <link name="imu_link">
@@ -82,4 +173,11 @@
       <material name="purple"/>
     </visual>
+    <collision>
+      <geometry><box size="0.06 0.03 0.05"/></geometry>
+    </collision>
+    <inertial>
+      <mass value="0.2"/>
+      <inertia ixx="0.001" ixy="0" ixz="0" iyy="0.001" iyz="0" izz="0.001"/>
+    </inertial>
   </link>
   <joint name="imu_joint" type="fixed">
@@ -88,3 +186,21 @@
     <origin xyz="0 0 0.095" rpy="1.57 0 0"/>
   </joint>
+  <gazebo reference="imu_link">
+    <sensor name="imu_sensor" type="imu">
+      <always_on>true</always_on>
+      <update_rate>100</update_rate>
+      <topic>imu/data</topic>
+      <imu>
+        <noise>
+          <type>gaussian</type>
+          <rate>
+            <mean>0.0</mean>
+            <stddev>0.0002</stddev>
+            <bias_mean>0.000007</bias_mean>
+            <bias_stddev>0.0000001</bias_stddev>
+          </rate>
+        </noise>
+      </imu>
+    </sensor>
+  </gazebo>
 </robot>

Commit message: MISC: Extracted ros2control block into a separate file

File: src/fourwd_robot/urdf/fourwd_robot.xacro (robot description, xacro)
@@ -10,4 +10,5 @@
   <xacro:property name="wheelbase"      value="0.36"/>
   <xacro:property name="track_width"    value="0.334"/>
+<xacro:include filename="$(find fourwd_robot)/urdf/robot.ros2control.xacro"/>
   <!-- ====================== MATERIALS ====================== -->
   <material name="blue">
@@ -119,32 +120,4 @@
   </plugin>
 </gazebo>
-  <!-- ====================== ROS2_CONTROL ====================== -->
-  <ros2_control name="fourwd_robot" type="system">
-     <hardware>
-        <!-- <plugin>mock_components/GenericSystem</plugin> -->
-        <plugin>gz_ros2_control/GazeboSimSystem</plugin>
-        <!-- <params name="calculate_dynamics">true</params> -->
-    </hardware>
-    <joint name="fl_wheel_joint">
-      <command_interface name="velocity"/>
-      <state_interface name="velocity"/>
-      <state_interface name="position"/>
-    </joint>
-    <joint name="fr_wheel_joint">
-      <command_interface name="velocity"/>
-      <state_interface name="velocity"/>
-      <state_interface name="position"/>
-    </joint>
-    <joint name="rl_wheel_joint">
-      <command_interface name="velocity"/>
-      <state_interface name="velocity"/>
-      <state_interface name="position"/>
-    </joint>
-    <joint name="rr_wheel_joint">
-      <command_interface name="velocity"/>
-      <state_interface name="velocity"/>
-      <state_interface name="position"/>
-    </joint>
-  </ros2_control>
    <!-- Gazebo LiDAR Plugin (GPU Ray Sensor) -->
   <gazebo reference="lidar_link">
@@ -212,3 +185,4 @@
     </sensor>
   </gazebo>
+<xacro:robot_ros2_control name="fourwd_robot" prefix=""/>
 </robot>
