Commit message: Proper naming used to import and use ros2control node in main xacro

File: src/fourwd_robot/urdf/robot.ros2control.xacro (robot description, xacro)
@@ -1,5 +1,5 @@
 <?xml version="1.0"?>
 <robot xmlns:xacro="http://www.ros.org/wiki/xacro">
-  <xacro:macro name="fourwd_robot" params="name prefix:=''">
+  <xacro:macro name="robot_ros2_control" params="name prefix:=''">
       <!-- ====================== ROS2_CONTROL ====================== -->
   <ros2_control name="${name}" type="system">
